File: _autosave-wireless_alice.kicad_sch (KiCad schematic)
At the start: 178 parts, among them J1 Conn_01x04, J2 Conn_01x02, J3 Conn_01x04, J4 Conn_01x02, J5 Conn_01x01, J6 Conn_01x01, J7 Conn_01x01, J8 Conn_01x01, Q1 AO3407, SW1 SW_SPDT, SW2 SW_Push, SW3 Rotary_Encoder_Switch, U1 E73-2G4M08S1C, U2 MCP73831, U3 AP2112K-3.3, U4 USBLC6-2SC6, X1 32768kHz

Commit message: more progress my guy
Parts:
- D10, D11, D12, D13, D14, D15, D16, D17, D18, D19, D2, D20, D21, D22, D23, D24, D25, D26, D27, D28, D29, D3, D30, D31, D32, D33, D34, D35, D36, D37, D38, D39, D4, D40, D41, D42, D43, D44, D45, D46, D47, D48, D49, D5, D50, D51, D52, D53, D54, D55, D56, D57, D58, D59, D6, D60, D61, D62, D63, D64, D65, D66, D67, D7, D8, D9: footprint Diode_THT:D_5W_P12.70mm_Horizontal -> Diode_SMD:D_SOD-123
- MX63: footprint Button_Switch_Keyboard:SW_Cherry_MX_1.00u_PCB -> yeye:SW_Cherry_MX_2.25u_PCB_Flipped
