File: wireless_alice.kicad_pcb (KiCad board)
At the start: 2 copper layers, 171 parts, among them J1 Conn_01x04, J2 Conn_01x02, J3 Conn_01x04, J4 Conn_01x02, J5 Conn_01x01, J6 Conn_01x01, J7 Conn_01x01, J8 Conn_01x01, Q1 AO3407, SW1 SW_SPDT, SW2 SW_Push, SW3 Rotary_Encoder_Switch, U1 E73-2G4M08S1C, U2 MCP73831, U3 AP2112K-3.3, U4 USBLC6-2SC6, X1 32768kHz

Commit message: More pcb refinement
Parts:
- MX1, MX10, MX11, MX12, MX13, MX14, MX15, MX16, MX18, MX19, MX2, MX20, MX21, MX22, MX23, MX24, MX25, MX27, MX28, MX29, MX3, MX30, MX31A1, MX32, MX33, MX34, MX35, MX36, MX37, MX39, MX4, MX40, MX42, MX43, MX44, MX45, MX46, MX47, MX48, MX49, MX51, MX52, MX53, MX54, MX55, MX56, MX57, MX58, MX59, MX59A2, MX60, MX62, MX62A2, MX9: footprint Button_Switch_Keyboard:SW_Cherry_MX_1.00u_Plate -> Button_Switch_Keyboard:SW_Cherry_MX_1.00u_PCB
- MX17, MX8: footprint Button_Switch_Keyboard:SW_Cherry_MX_1.50u_Plate -> Button_Switch_Keyboard:SW_Cherry_MX_1.50u_PCB
- MX26: footprint Button_Switch_Keyboard:SW_Cherry_MX_2.25u_Plate -> Button_Switch_Keyboard:SW_Cherry_MX_2.25u_PCB
- MX26A1, MX59A1: footprint Button_Switch_Keyboard:SW_Cherry_MX_2.00u_Plate -> Button_Switch_Keyboard:SW_Cherry_MX_2.00u_PCB
- MX31: footprint Button_Switch_Keyboard:SW_Cherry_MX_1.25u_Plate -> Button_Switch_Keyboard:SW_Cherry_MX_1.25u_PCB
- MX38: footprint Button_Switch_Keyboard:SW_Cherry_MX_1.00u_Plate -> Button_Switch_Keyboard:SW_Cherry_MX_1.00u_PCB; moved to B.Cu
- MX41: footprint Button_Switch_Keyboard:SW_Cherry_MX_2.75u_Plate -> Button_Switch_Keyboard:SW_Cherry_MX_2.75u_PCB
- MX5: footprint Button_Switch_Keyboard:SW_Cherry_MX_1.00u_Plate -> Button_Switch_Keyboard:SW_Cherry_MX_1.50u_PCB
- MX6, MX6A1: footprint Button_Switch_Keyboard:SW_Cherry_MX_1.00u_Plate -> Button_Switch_Keyboard:SW_Cherry_MX_1.75u_PCB
- MX61: footprint Button_Switch_Keyboard:SW_Cherry_MX_1.75u_Plate -> Button_Switch_Keyboard:SW_Cherry_MX_2.75u_PCB
- MX62A1: footprint Button_Switch_Keyboard:SW_Cherry_MX_2.75u_PCB -> Button_Switch_Keyboard:SW_Cherry_MX_1.75u_PCB
- MX63: footprint Button_Switch_Keyboard:SW_Cherry_MX_1.00u_Plate -> yeye:SW_Cherry_MX_2.25u_PCB_Flipped
- MX7: footprint Button_Switch_Keyboard:SW_Cherry_MX_1.00u_Plate -> Button_Switch_Keyboard:SW_Cherry_MX_2.75u_PCB
- moved MX62A1 670.3 mm to (610.7, 168.2)
- moved MX61 665.0 mm to (620.2, 168.2)
- moved MX64 647.9 mm to (628.4, 187.3)
- moved MX41 620.9 mm to (508.2, 196.4), turned to 12 degrees
- moved MX59A1 604.4 mm to (612.2, 116.1)
- moved MX62A2 591.6 mm to (636.9, 168.2)
- moved MX53 571.8 mm to (570.8, 149.2)
- moved MX58 566.1 mm to (584.5, 168.2)
- moved MX50 561.3 mm to (548.6, 189.3), turned to 12 degrees
- moved MX63 551.6 mm to (620.8, 149.2)
- moved MX54 550.3 mm to (565.4, 168.2)
- moved MX44 549.7 mm to (530.6, 152.7), turned to 12 degrees
- moved MX59A2 547.0 mm to (624.3, 111.1)
- moved MX57 543.9 mm to (589.9, 149.2)
- moved MX52 540.7 mm to (562.2, 129.1)
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Connections:
- J2 pad 1: VBAT -> VBATT

Commit message: more progress my guy
Parts:
- D10, D11, D12, D13, D14, D15, D16, D17, D18, D19, D2, D20, D21, D22, D23, D24, D25, D26, D27, D28, D29, D3, D30, D31, D32, D33, D34, D35, D36, D37, D38, D39, D4, D40, D41, D42, D43, D44, D45, D46, D47, D48, D49, D5, D50, D51, D52, D53, D54, D55, D56, D57, D58, D59, D6, D60, D61, D62, D63, D64, D65, D66, D67, D7, D8, D9: footprint Diode_THT:D_5W_P12.70mm_Horizontal -> Diode_SMD:D_SOD-123
- moved D59 434.6 mm to (577.3, 179.6)
- moved D67 429.9 mm to (628.1, 197.4)
- moved D66 425.1 mm to (635.7, 177.1)
- moved D31 423.3 mm to (457.9, 192.3)
- moved D64 409.0 mm to (620.5, 141.5)
- moved D62 404.5 mm to (613.7, 177.1)
- moved D22 404.3 mm to (419.5, 187.3)
- moved D51 400.2 mm to (541.7, 202.5)
- moved D48 393.8 mm to (536.6, 141.5)
- moved D42 393.4 mm to (506.8, 207.6)
- moved D18 393.3 mm to (402.0, 202.5)
- moved D28 391.8 mm to (445.2, 131.4)
- moved D9 390.0 mm to (348.7, 197.4)
- moved D65 388.2 mm to (617.9, 159.3)
- moved SW3 386.8 mm to (320.8, 121.2), turned to 90 degrees
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