File: wireless_alice.kicad_sch (KiCad schematic)
At the start: 178 parts, among them J1 Conn_01x04, J2 Conn_01x02, J3 Conn_01x04, J4 Conn_01x02, J5 Conn_01x01, J6 Conn_01x01, J7 Conn_01x01, J8 Conn_01x01, Q1 AO3407, SW1 SW_SPDT, SW2 SW_Push, SW3 Rotary_Encoder_Switch, U1 E73-2G4M08S1C, U2 MCP73831, U3 AP2112K-3.3, U4 USBLC6-2SC6, X1 32768kHz

Commit message: More pcb refinement
Parts:
- MX1, MX10, MX11, MX12, MX13, MX14, MX15, MX16, MX18, MX19, MX2, MX20, MX21, MX22, MX23, MX24, MX25, MX27, MX28, MX29, MX3, MX30, MX31A1, MX32, MX33, MX34, MX35, MX36, MX37, MX38, MX39, MX4, MX40, MX42, MX43, MX44, MX45, MX46, MX47, MX48, MX49, MX5, MX51, MX52, MX53, MX54, MX55, MX56, MX57, MX58, MX59, MX59A2, MX60, MX62, MX62A2, MX63, MX9: footprint Button_Switch_Keyboard:SW_Cherry_MX_1.00u_Plate -> Button_Switch_Keyboard:SW_Cherry_MX_1.00u_PCB
- MX17, MX8: footprint Button_Switch_Keyboard:SW_Cherry_MX_1.50u_Plate -> Button_Switch_Keyboard:SW_Cherry_MX_1.50u_PCB
- MX26: footprint Button_Switch_Keyboard:SW_Cherry_MX_2.25u_Plate -> Button_Switch_Keyboard:SW_Cherry_MX_2.25u_PCB
- MX26A1, MX59A1: footprint Button_Switch_Keyboard:SW_Cherry_MX_2.00u_Plate -> Button_Switch_Keyboard:SW_Cherry_MX_2.00u_PCB
- MX31: footprint Button_Switch_Keyboard:SW_Cherry_MX_1.25u_Plate -> Button_Switch_Keyboard:SW_Cherry_MX_1.25u_PCB
- MX41: footprint Button_Switch_Keyboard:SW_Cherry_MX_2.75u_Plate -> Button_Switch_Keyboard:SW_Cherry_MX_2.75u_PCB
- MX6, MX6A1: footprint Button_Switch_Keyboard:SW_Cherry_MX_1.00u_Plate -> Button_Switch_Keyboard:SW_Cherry_MX_1.75u_PCB
- MX61: footprint Button_Switch_Keyboard:SW_Cherry_MX_1.75u_Plate -> Button_Switch_Keyboard:SW_Cherry_MX_1.75u_PCB
- MX7: footprint Button_Switch_Keyboard:SW_Cherry_MX_1.00u_Plate -> Button_Switch_Keyboard:SW_Cherry_MX_2.75u_PCB
Connections:
- net VBAT: no longer J2.1 (Pin_1)
- net VBATT: now also J2.1 (Pin_1)

Commit message: more progress my guy
Parts:
- MX5: footprint Button_Switch_Keyboard:SW_Cherry_MX_1.00u_PCB -> Button_Switch_Keyboard:SW_Cherry_MX_1.50u_PCB
- MX61: footprint Button_Switch_Keyboard:SW_Cherry_MX_1.75u_PCB -> Button_Switch_Keyboard:SW_Cherry_MX_2.75u_PCB
- MX62A1: footprint Button_Switch_Keyboard:SW_Cherry_MX_2.75u_PCB -> Button_Switch_Keyboard:SW_Cherry_MX_1.75u_PCB
- MX63: footprint Button_Switch_Keyboard:SW_Cherry_MX_1.00u_PCB -> yeye:SW_Cherry_MX_2.25u_PCB_Flipped
Changed lines of the file:
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@@
       (effects (font (size 0.508 0.508)))
     )
-    (property "Footprint" "Button_Switch_Keyboard:SW_Cherry_MX_1.00u_PCB" (id 2) (at 377.825 156.845 0)
+    (property "Footprint" "yeye:SW_Cherry_MX_2.25u_PCB_Flipped" (id 2) (at 377.825 156.845 0)
       (effects (font (size 1.524 1.524)) hide)
     )
@@
       (effects (font (size 0.508 0.508)))
     )
-    (property "Footprint" "Button_Switch_Keyboard:SW_Cherry_MX_1.00u_PCB" (id 2) (at 127.635 133.985 0)
+    (property "Footprint" "Button_Switch_Keyboard:SW_Cherry_MX_1.50u_PCB" (id 2) (at 127.635 133.985 0)
       (effects (font (size 1.524 1.524)) hide)
     )
@@
       (effects (font (size 0.508 0.508)))
     )
-    (property "Footprint" "Button_Switch_Keyboard:SW_Cherry_MX_2.75u_PCB" (id 2) (at 360.045 179.705 0)
+    (property "Footprint" "Button_Switch_Keyboard:SW_Cherry_MX_1.75u_PCB" (id 2) (at 360.045 179.705 0)
       (effects (font (size 1.524 1.524)) hide)
     )
@@
       (effects (font (size 0.508 0.508)))
     )
-    (property "Footprint" "Button_Switch_Keyboard:SW_Cherry_MX_1.75u_PCB" (id 2) (at 361.315 180.975 0)
+    (property "Footprint" "Button_Switch_Keyboard:SW_Cherry_MX_2.75u_PCB" (id 2) (at 361.315 180.975 0)
       (effects (font (size 1.524 1.524)) hide)
     )
@@
     )
     (path "/687a989c-2739-4b69-8c5b-8b9ab4b489fd"
-      (reference "MX5") (unit 1) (value "MX-NoLED") (footprint "Button_Switch_Keyboard:SW_Cherry_MX_1.00u_PCB")
+      (reference "MX5") (unit 1) (value "MX-NoLED") (footprint "Button_Switch_Keyboard:SW_Cherry_MX_1.50u_PCB")
     )
     (path "/ff939585-5e0a-465d-b32b-de7b8cc8a32a"
@@
     )
     (path "/d4f1d07e-6b45-4bbf-a257-6e89fccb808c"
-      (reference "MX61") (unit 1) (value "MX-NoLED") (footprint "Button_Switch_Keyboard:SW_Cherry_MX_1.75u_PCB")
+      (reference "MX61") (unit 1) (value "MX-NoLED") (footprint "Button_Switch_Keyboard:SW_Cherry_MX_2.75u_PCB")
     )
     (path "/1006cd0b-337b-4242-baa4-93d9ca4e4554"
@@
     )
     (path "/9a06ce17-9699-412c-bb48-ad3e933713c1"
-      (reference "MX62A1") (unit 1) (value "MX-NoLED") (footprint "Button_Switch_Keyboard:SW_Cherry_MX_2.75u_PCB")
+      (reference "MX62A1") (unit 1) (value "MX-NoLED") (footprint "Button_Switch_Keyboard:SW_Cherry_MX_1.75u_PCB")
     )
     (path "/67f821c6-9856-4a62-b9ed-081569ce84f5"
@@
     )
     (path "/1db58005-d85d-46fc-9246-2aa60e8872e8"
-      (reference "MX63") (unit 1) (value "MX-NoLED") (footprint "Button_Switch_Keyboard:SW_Cherry_MX_1.00u_PCB")
+      (reference "MX63") (unit 1) (value "MX-NoLED") (footprint "yeye:SW_Cherry_MX_2.25u_PCB_Flipped")
     )
     (path "/744dee25-d236-49b7-a100-a996af94024c"
